Commit message: working camera stream and display

File: mad_bot/model/mad_bot.urdf (robot description, URDF)
Before this commit: robot mad_bot, 3 links, 2 joints
Links:
- added link camera_link, mass 0.1; collision box size=0.1 0.1 0.05; visual box size=0.1 0.1 0.05
- added link caster_back, mass 1; collision sphere radius=0.075; visual sphere radius=0.075
- added link caster_front, mass 1; collision sphere radius=0.075; visual sphere radius=0.075
Joints:
- added joint back_caster_joint: type ball, parent chassis, child caster_back, origin xyz=0.4 0 -0.275 rpy=0 0 0
- added joint camera_joint: type fixed, parent chassis, child camera_link, origin xyz=0.3 0 0.225 rpy=0 0 0
- added joint front_caster_joint: type ball, parent chassis, child caster_front, origin xyz=-0.4 0 -0.275 rpy=0 0 0
- joint left_wheel_joint: limit lower=-1000 upper=1000 effort=10 velocity=0 -> lower=-1000 upper=1000 effort=10; origin (none) -> xyz=0 0.325 0 rpy=0 0 0
- joint right_wheel_joint: limit lower=-1000 upper=1000 effort=10 velocity=0 -> lower=-1000 upper=1000 effort=10; origin (none) -> xyz=0 -0.325 0 rpy=0 0 0
